Commit message: add

File: husky_gazebo/urdf/accessories/kinect_camera.gazebo.xacro (robot description, xacro)
@@ -3,5 +3,5 @@
 <xacro:macro name="kinect_camera_gazebo" params="prefix">
   <joint name="${prefix}_optical_joint" type="fixed">
-    <origin xyz="0 0 0" rpy="-1.5708 0 -1.5708"/>
+    <origin xyz="0 0 0" rpy="-1.5708  0 -1.5708"/>
     <parent link="${prefix}_link"/>
     <child link="${prefix}_frame_optical"/>
@@ -13,5 +13,5 @@
       <update_rate>20.0</update_rate>
       <camera>
-        <horizontal_fov>${60.0*M_PI/180.0}</horizontal_fov>
+        <horizontal_fov>${90.0*M_PI/180.0}</horizontal_fov>
         <image>
           <format>R8G8B8</format>
@@ -24,5 +24,5 @@
         </clip>
       </camera>
-      <plugin name="kinect_${prefix}_controller" filename="libgazebo_ros_openni_kinect.so">
+      <plugin name="kinect_${prefix}_controller" filename="libkinectplugin.so">
         <cameraName>${prefix}</cameraName>
         <alwaysOn>true</alwaysOn>

File: husky_gazebo/urdf/description2.gazebo.xacro (robot description, xacro)
@@ -24,6 +24,6 @@
   <xacro:arg name="laser_enabled" default="true" />
   <xacro:arg name="ur5_enabled" default="false" />
-  <xacro:arg name="kinect_enabled" default="true" />
-  <xacro:include filename="$(find husky_description)/urdf/husky.urdf.xacro" />
+  <xacro:arg name="kinect_enabled" default="false" />
+  <xacro:include filename="$(find husky_description)/urdf/husky2.urdf.xacro" />
   <xacro:include filename="$(find husky_gazebo)/urdf/husky.gazebo.xacro" />
   <!-- Gazebo plugin for ROS Control -->

File: husky_gazebo/urdf/description3.gazebo.xacro (robot description, xacro)
@@ -24,6 +24,6 @@
   <xacro:arg name="laser_enabled" default="true" />
   <xacro:arg name="ur5_enabled" default="false" />
-  <xacro:arg name="kinect_enabled" default="true" />
-  <xacro:include filename="$(find husky_description)/urdf/husky.urdf.xacro" />
+  <xacro:arg name="kinect_enabled" default="false" />
+  <xacro:include filename="$(find husky_description)/urdf/husky3.urdf.xacro" />
   <xacro:include filename="$(find husky_gazebo)/urdf/husky.gazebo.xacro" />
   <!-- Gazebo plugin for ROS Control -->

File: husky_gazebo/urdf/husky.gazebo.xacro (robot description, xacro)
@@ -52,4 +52,14 @@
         <drift>0.0001 0.0001 0.0001</drift>
       </plugin>
+    <plugin name="p3d_base_controller" filename="libgazebo_ros_p3d.so">
+      <alwaysOn>true</alwaysOn>
+      <updateRate>50.0</updateRate>
+      <bodyName>base_link</bodyName>
+      <topicName>ground_truth/state</topicName>
+      <gaussianNoise>0.01</gaussianNoise>
+      <frameName>world</frameName>
+      <xyzOffsets>0 0 0</xyzOffsets>
+      <rpyOffsets>0 0 0</rpyOffsets>
+    </plugin>
     </gazebo>
     <xacro:if value="$(arg ur5_enabled)">

Commit message: add

File: husky_gazebo/urdf/accessories/kinect_camera.gazebo.xacro (robot description, xacro)
@@ -3,5 +3,5 @@
 <xacro:macro name="kinect_camera_gazebo" params="prefix">
   <joint name="${prefix}_optical_joint" type="fixed">
-    <origin xyz="0 0 0" rpy="-1.5708  0 -1.5708"/>
+    <origin xyz="0 0 0" rpy="-1.5708 0 -1.5708"/>
     <parent link="${prefix}_link"/>
     <child link="${prefix}_frame_optical"/>
@@ -13,5 +13,5 @@
       <update_rate>20.0</update_rate>
       <camera>
-        <horizontal_fov>${90.0*M_PI/180.0}</horizontal_fov>
+        <horizontal_fov>${60.0*M_PI/180.0}</horizontal_fov>
         <image>
           <format>R8G8B8</format>
@@ -24,5 +24,5 @@
         </clip>
       </camera>
-      <plugin name="kinect_${prefix}_controller" filename="libkinectplugin.so">
+      <plugin name="kinect_${prefix}_controller" filename="libgazebo_ros_openni_kinect.so">
         <cameraName>${prefix}</cameraName>
         <alwaysOn>true</alwaysOn>

File: husky_gazebo/urdf/description.gazebo.xacro (robot description, xacro)
@@ -24,5 +24,5 @@
   <xacro:arg name="laser_enabled" default="true" />
   <xacro:arg name="ur5_enabled" default="false" />
-  <xacro:arg name="kinect_enabled" default="true" />
+  <xacro:arg name="kinect_enabled" default="false" />
   <xacro:include filename="$(find husky_description)/urdf/husky.urdf.xacro" />
   <xacro:include filename="$(find husky_gazebo)/urdf/husky.gazebo.xacro" />

File: husky_gazebo/urdf/husky.gazebo.xacro (robot description, xacro)
@@ -52,14 +52,4 @@
         <drift>0.0001 0.0001 0.0001</drift>
       </plugin>
-    <plugin name="p3d_base_controller" filename="libgazebo_ros_p3d.so">
-      <alwaysOn>true</alwaysOn>
-      <updateRate>50.0</updateRate>
-      <bodyName>base_link</bodyName>
-      <topicName>ground_truth/state</topicName>
-      <gaussianNoise>0.01</gaussianNoise>
-      <frameName>world</frameName>
-      <xyzOffsets>0 0 0</xyzOffsets>
-      <rpyOffsets>0 0 0</rpyOffsets>
-    </plugin>
     </gazebo>
     <xacro:if value="$(arg ur5_enabled)">
